Commit message: xacro pointing to ros package

File: urdf/leg.xacro (robot description, xacro)
@@ -50,5 +50,5 @@
                     <origin xyz="0.01950 0 0" rpy="0 0 0" />
                     <geometry>
-                        <mesh filename="package:///solo12_description/meshes/${mesh_ext}/solo12/solo12_hip_fe_fl.${mesh_ext}"/>
+                      <mesh filename="package://solo12_description/meshes/collision/hip_fe_fl.${mesh_ext}"/>
                     </geometry>
                 </xacro:if>
@@ -56,5 +56,5 @@
                     <origin xyz="-0.01950 0 0" rpy="0 0 0" />
                     <geometry>
-                        <mesh filename="package://robot_properties_solo/resources/meshes/${mesh_ext}/solo12/solo12_hip_fe_hl.${mesh_ext}"/>
+                      <mesh filename="package://solo12_description/meshes/collision/hip_fe_hl.${mesh_ext}"/>
                     </geometry>
                 </xacro:unless>
@@ -64,5 +64,5 @@
                     <origin xyz="0.01950 0 0" rpy="0 0 0" />
                     <geometry>
-                        <mesh filename="package://robot_properties_solo/resources/meshes/${mesh_ext}/solo12/solo12_hip_fe_fr.${mesh_ext}"/>
+                        <mesh filename="package://solo12_description/meshes/collision/hip_fe_fr.${mesh_ext}"/>
                     </geometry>
                 </xacro:if>
@@ -70,5 +70,5 @@
                     <origin xyz="-0.01950 0 0" rpy="0 0 0" />
                     <geometry>
-                        <mesh filename="package://robot_properties_solo/resources/meshes/${mesh_ext}/solo12/solo12_hip_fe_hr.${mesh_ext}"/>
+                        <mesh filename="package://solo12_description/meshes/collision/hip_fe_hr.${mesh_ext}"/>
                     </geometry>
                 </xacro:unless>
@@ -84,5 +84,5 @@
                     <origin xyz="0.01950 0 0" rpy="0 0 0" />
                     <geometry>
-                        <mesh filename="package://robot_properties_solo/resources/meshes/${mesh_ext}/solo12/solo12_hip_fe_fl.${mesh_ext}"/>
+                        <mesh filename="package://solo12_description/meshes/collision/hip_fe_fl.${mesh_ext}"/>
                     </geometry>
                 </xacro:if>
@@ -90,5 +90,5 @@
                     <origin xyz="-0.01950 0 0" rpy="0 0 0" />
                     <geometry>
-                        <mesh filename="package://robot_properties_solo/resources/meshes/${mesh_ext}/solo12/solo12_hip_fe_hl.${mesh_ext}"/>
+                      <mesh filename="package://solo12_description/meshes/collision/hip_fe_hl.${mesh_ext}"/>
                     </geometry>
                 </xacro:unless>
@@ -98,5 +98,5 @@
                     <origin xyz="0.01950 0 0" rpy="0 0 0" />
                     <geometry>
-                        <mesh filename="package://robot_properties_solo/resources/meshes/${mesh_ext}/solo12/solo12_hip_fe_fr.${mesh_ext}"/>
+                        <mesh filename="package://solo12_description/meshes/collision/hip_fe_fr.${mesh_ext}"/>
                     </geometry>
                 </xacro:if>
@@ -104,5 +104,5 @@
                     <origin xyz="-0.01950 0 0" rpy="0 0 0" />
                     <geometry>
-                        <mesh filename="package://robot_properties_solo/resources/meshes/${mesh_ext}/solo12/solo12_hip_fe_hr.${mesh_ext}"/>
+                        <mesh filename="package://solo12_description/meshes/collision/hip_fe_hr.${mesh_ext}"/>
                     </geometry>
                 </xacro:unless>
@@ -231,8 +231,8 @@
         <geometry>
           <xacro:unless value="${is_right}">
-            <mesh filename="package://robot_properties_solo/resources/meshes/${mesh_ext}/without_foot/solo_upper_leg_left_side.${mesh_ext}"/>
-          </xacro:unless>
-          <xacro:if value="${is_right}">
-            <mesh filename="package://robot_properties_solo/resources/meshes/${mesh_ext}/without_foot/solo_upper_leg_right_side.${mesh_ext}"/>
+            <mesh filename="package://solo12_description/meshes/collision/isolated_upper_leg_left_side.${mesh_ext}"/>
+          </xacro:unless>
+          <xacro:if value="${is_right}">
+            <mesh filename="package://solo12_description/meshes/collision/isolated_upper_leg_right_side.${mesh_ext}"/>
           </xacro:if>
         </geometry>
@@ -246,8 +246,8 @@
         <geometry>
           <xacro:unless value="${is_right}">
-            <mesh filename="package://robot_properties_solo/resources/meshes/${mesh_ext}/without_foot/solo_upper_leg_left_side.${mesh_ext}"/>
-          </xacro:unless>
-          <xacro:if value="${is_right}">
-            <mesh filename="package://robot_properties_solo/resources/meshes/${mesh_ext}/without_foot/solo_upper_leg_right_side.${mesh_ext}"/>
+            <mesh filename="package://solo12_description/meshes/collision/isolated_upper_leg_left_side.${mesh_ext}"/>
+          </xacro:unless>
+          <xacro:if value="${is_right}">
+            <mesh filename="package://solo12_description/meshes/collision/isolated_upper_leg_right_side.${mesh_ext}"/>
           </xacro:if>
         </geometry>
@@ -316,8 +316,8 @@
         <geometry>
           <xacro:unless value="${is_right}">
-            <mesh filename="package://robot_properties_solo/resources/meshes/${mesh_ext}/without_foot/solo_lower_leg_v2_left_side.${mesh_ext}"/>
-          </xacro:unless>
-          <xacro:if value="${is_right}">
-            <mesh filename="package://robot_properties_solo/resources/meshes/${mesh_ext}/without_foot/solo_lower_leg_v2_right_side.${mesh_ext}"/>
+            <mesh filename="package://solo12_description/meshes/collision/isolated_lower_leg_v2_left_side.${mesh_ext}"/>
+          </xacro:unless>
+          <xacro:if value="${is_right}">
+            <mesh filename="package://solo12_description/meshes/collision/isolated_lower_leg_v2_right_side.${mesh_ext}"/>
           </xacro:if>
         </geometry>
@@ -331,8 +331,8 @@
         <geometry>
           <xacro:unless value="${is_right}">
-            <mesh filename="package://robot_properties_solo/resources/meshes/${mesh_ext}/without_foot/solo_lower_leg_v2_left_side.${mesh_ext}"/>
-          </xacro:unless>
-          <xacro:if value="${is_right}">
-            <mesh filename="package://robot_properties_solo/resources/meshes/${mesh_ext}/without_foot/solo_lower_leg_v2_right_side.${mesh_ext}"/>
+            <mesh filename="package://solo12_description/meshes/collision/isolated_lower_leg_v2_left_side.${mesh_ext}"/>
+          </xacro:unless>
+          <xacro:if value="${is_right}">
+            <mesh filename="package://solo12_description/meshes/collision/isolated_lower_leg_v2_right_side.${mesh_ext}"/>
           </xacro:if>
         </geometry>

File: urdf/solo12.urdf.xacro (robot description, xacro)
@@ -25,5 +25,5 @@
         <origin xyz="0 0 0" rpy="0 0 0" />
         <geometry>
-          <mesh filename="package://robot_properties_solo/resources/meshes/${mesh_ext}/solo12/solo_12_base.${mesh_ext}"/>
+          <mesh filename="package://solo12_description/meshes/collision/base.${mesh_ext}"/>
         </geometry>
         <material name="${color_name}">
@@ -35,5 +35,5 @@
         <origin xyz="0 0 0" rpy="0 0 0" />
         <geometry>
-          <mesh filename="package://robot_properties_solo/resources/meshes/${mesh_ext}/solo12/solo_12_base.${mesh_ext}"/>
+          <mesh filename="package://solo12_description/meshes/collision/base.${mesh_ext}"/>
         </geometry>
         <material name="${color_name}">

Commit message: fix model spawn in gazebo

File: urdf/leg.xacro (robot description, xacro)
@@ -50,5 +50,5 @@
                     <origin xyz="0.01950 0 0" rpy="0 0 0" />
                     <geometry>
-                      <mesh filename="package://solo12_description/meshes/collision/hip_fe_fl.${mesh_ext}"/>
+              <mesh filename="file://$(find solo12_description)/meshes/collision/hip_fe_fl.${mesh_ext}"/>
                     </geometry>
                 </xacro:if>
@@ -56,5 +56,5 @@
                     <origin xyz="-0.01950 0 0" rpy="0 0 0" />
                     <geometry>
-                      <mesh filename="package://solo12_description/meshes/collision/hip_fe_hl.${mesh_ext}"/>
+                      <mesh filename="file://$(find solo12_description)/meshes/collision/hip_fe_hl.${mesh_ext}"/>
                     </geometry>
                 </xacro:unless>
@@ -64,5 +64,5 @@
                     <origin xyz="0.01950 0 0" rpy="0 0 0" />
                     <geometry>
-                        <mesh filename="package://solo12_description/meshes/collision/hip_fe_fr.${mesh_ext}"/>
+                        <mesh filename="file://$(find solo12_description)/meshes/collision/hip_fe_fr.${mesh_ext}"/>
                     </geometry>
                 </xacro:if>
@@ -70,5 +70,5 @@
                     <origin xyz="-0.01950 0 0" rpy="0 0 0" />
                     <geometry>
-                        <mesh filename="package://solo12_description/meshes/collision/hip_fe_hr.${mesh_ext}"/>
+                        <mesh filename="file://$(find solo12_description)/meshes/collision/hip_fe_hr.${mesh_ext}"/>
                     </geometry>
                 </xacro:unless>
@@ -84,5 +84,5 @@
                     <origin xyz="0.01950 0 0" rpy="0 0 0" />
                     <geometry>
-                        <mesh filename="package://solo12_description/meshes/collision/hip_fe_fl.${mesh_ext}"/>
+                        <mesh filename="file://$(find solo12_description)/meshes/collision/hip_fe_fl.${mesh_ext}"/>
                     </geometry>
                 </xacro:if>
@@ -90,5 +90,5 @@
                     <origin xyz="-0.01950 0 0" rpy="0 0 0" />
                     <geometry>
-                      <mesh filename="package://solo12_description/meshes/collision/hip_fe_hl.${mesh_ext}"/>
+                      <mesh filename="file://$(find solo12_description)/meshes/collision/hip_fe_hl.${mesh_ext}"/>
                     </geometry>
                 </xacro:unless>
@@ -98,5 +98,5 @@
                     <origin xyz="0.01950 0 0" rpy="0 0 0" />
                     <geometry>
-                        <mesh filename="package://solo12_description/meshes/collision/hip_fe_fr.${mesh_ext}"/>
+                        <mesh filename="file://$(find solo12_description)/meshes/collision/hip_fe_fr.${mesh_ext}"/>
                     </geometry>
                 </xacro:if>
@@ -104,5 +104,5 @@
                     <origin xyz="-0.01950 0 0" rpy="0 0 0" />
                     <geometry>
-                        <mesh filename="package://solo12_description/meshes/collision/hip_fe_hr.${mesh_ext}"/>
+                        <mesh filename="file://$(find solo12_description)/meshes/collision/hip_fe_hr.${mesh_ext}"/>
                     </geometry>
                 </xacro:unless>
@@ -231,8 +231,8 @@
         <geometry>
           <xacro:unless value="${is_right}">
-            <mesh filename="package://solo12_description/meshes/collision/isolated_upper_leg_left_side.${mesh_ext}"/>
-          </xacro:unless>
-          <xacro:if value="${is_right}">
-            <mesh filename="package://solo12_description/meshes/collision/isolated_upper_leg_right_side.${mesh_ext}"/>
+            <mesh filename="file://$(find solo12_description)/meshes/collision/isolated_upper_leg_left_side.${mesh_ext}"/>
+          </xacro:unless>
+          <xacro:if value="${is_right}">
+            <mesh filename="file://$(find solo12_description)/meshes/collision/isolated_upper_leg_right_side.${mesh_ext}"/>
           </xacro:if>
         </geometry>
@@ -246,8 +246,8 @@
         <geometry>
           <xacro:unless value="${is_right}">
-            <mesh filename="package://solo12_description/meshes/collision/isolated_upper_leg_left_side.${mesh_ext}"/>
-          </xacro:unless>
-          <xacro:if value="${is_right}">
-            <mesh filename="package://solo12_description/meshes/collision/isolated_upper_leg_right_side.${mesh_ext}"/>
+            <mesh filename="file://$(find solo12_description)/meshes/collision/isolated_upper_leg_left_side.${mesh_ext}"/>
+          </xacro:unless>
+          <xacro:if value="${is_right}">
+            <mesh filename="file://$(find solo12_description)/meshes/collision/isolated_upper_leg_right_side.${mesh_ext}"/>
           </xacro:if>
         </geometry>
@@ -316,8 +316,8 @@
         <geometry>
           <xacro:unless value="${is_right}">
-            <mesh filename="package://solo12_description/meshes/collision/isolated_lower_leg_v2_left_side.${mesh_ext}"/>
-          </xacro:unless>
-          <xacro:if value="${is_right}">
-            <mesh filename="package://solo12_description/meshes/collision/isolated_lower_leg_v2_right_side.${mesh_ext}"/>
+            <mesh filename="file://$(find solo12_description)/meshes/collision/isolated_lower_leg_v2_left_side.${mesh_ext}"/>
+          </xacro:unless>
+          <xacro:if value="${is_right}">
+            <mesh filename="file://$(find solo12_description)/meshes/collision/isolated_lower_leg_v2_right_side.${mesh_ext}"/>
           </xacro:if>
         </geometry>
@@ -331,8 +331,8 @@
         <geometry>
           <xacro:unless value="${is_right}">
-            <mesh filename="package://solo12_description/meshes/collision/isolated_lower_leg_v2_left_side.${mesh_ext}"/>
-          </xacro:unless>
-          <xacro:if value="${is_right}">
-            <mesh filename="package://solo12_description/meshes/collision/isolated_lower_leg_v2_right_side.${mesh_ext}"/>
+            <mesh filename="file://$(find solo12_description)/meshes/collision/isolated_lower_leg_v2_left_side.${mesh_ext}"/>
+          </xacro:unless>
+          <xacro:if value="${is_right}">
+            <mesh filename="file://$(find solo12_description)/meshes/collision/isolated_lower_leg_v2_right_side.${mesh_ext}"/>
           </xacro:if>
         </geometry>
@@ -369,8 +369,8 @@
       <inertial>
         <origin xyz="0 0 0" rpy="0 0 0" />
-        <mass value="0.0"/>
-        <inertia ixx="0.0" ixy="0.0" ixz="0.0"
-                           iyy="0.0" iyz="0.0"
-                                     izz="0.0"/>
+        <mass value="0.01"/>
+        <inertia ixx="0.002" ixy="0.0" ixz="0.0"
+                           iyy="0.002" iyz="0.0"
+                                     izz="0.002"/>
       </inertial>
     </link> <!-- END FOOT LINK -->

File: urdf/solo12.urdf.xacro (robot description, xacro)
@@ -25,5 +25,6 @@
         <origin xyz="0 0 0" rpy="0 0 0" />
         <geometry>
-          <mesh filename="package://solo12_description/meshes/collision/base.${mesh_ext}"/>
+      <!-- <box size="0.1 0.1 0.1"/>-->
+      <mesh filename="file://$(find solo12_description)/meshes/collision/base.${mesh_ext}"/>
         </geometry>
         <material name="${color_name}">
@@ -35,5 +36,5 @@
         <origin xyz="0 0 0" rpy="0 0 0" />
         <geometry>
-          <mesh filename="package://solo12_description/meshes/collision/base.${mesh_ext}"/>
+      <mesh filename="file://$(find solo12_description)/meshes/collision/base.${mesh_ext}"/>
         </geometry>
         <material name="${color_name}">
