Commit message: Working Gazebo Plugin Control

File: solo12_description/urdf/modified/leg.xacro (robot description, xacro)
@@ -50,5 +50,5 @@
                     <origin xyz="0.01950 0 0" rpy="0 0 0" />
                     <geometry>
-              <mesh filename="file:///home/pratik/nala/gazebo_standalone/solo12_robot/solo12_description/meshes/collision/hip_fe_fl.${mesh_ext}"/>
+              <mesh filename="file:///home/pratik/Music/sdp/solo12_robot/solo12_description/meshes/collision/hip_fe_fl.${mesh_ext}"/>
                     </geometry>
                 </xacro:if>
@@ -56,5 +56,5 @@
                     <origin xyz="-0.01950 0 0" rpy="0 0 0" />
                     <geometry>
-                      <mesh filename="file:///home/pratik/nala/gazebo_standalone/solo12_robot/solo12_description/meshes/collision/hip_fe_hl.${mesh_ext}"/>
+                      <mesh filename="file:///home/pratik/Music/sdp/solo12_robot/solo12_description/meshes/collision/hip_fe_hl.${mesh_ext}"/>
                     </geometry>
                 </xacro:unless>
@@ -64,5 +64,5 @@
                     <origin xyz="0.01950 0 0" rpy="0 0 0" />
                     <geometry>
-                        <mesh filename="file:///home/pratik/nala/gazebo_standalone/solo12_robot/solo12_description/meshes/collision/hip_fe_fr.${mesh_ext}"/>
+                        <mesh filename="file:///home/pratik/Music/sdp/solo12_robot/solo12_description/meshes/collision/hip_fe_fr.${mesh_ext}"/>
                     </geometry>
                 </xacro:if>
@@ -70,5 +70,5 @@
                     <origin xyz="-0.01950 0 0" rpy="0 0 0" />
                     <geometry>
-                        <mesh filename="file:///home/pratik/nala/gazebo_standalone/solo12_robot/solo12_description/meshes/collision/hip_fe_hr.${mesh_ext}"/>
+                        <mesh filename="file:///home/pratik/Music/sdp/solo12_robot/solo12_description/meshes/collision/hip_fe_hr.${mesh_ext}"/>
                     </geometry>
                 </xacro:unless>
@@ -84,5 +84,5 @@
                     <origin xyz="0.01950 0 0" rpy="0 0 0" />
                     <geometry>
-                        <mesh filename="file:///home/pratik/nala/gazebo_standalone/solo12_robot/solo12_description/meshes/collision/hip_fe_fl.${mesh_ext}"/>
+                        <mesh filename="file:///home/pratik/Music/sdp/solo12_robot/solo12_description/meshes/collision/hip_fe_fl.${mesh_ext}"/>
                     </geometry>
                 </xacro:if>
@@ -90,5 +90,5 @@
                     <origin xyz="-0.01950 0 0" rpy="0 0 0" />
                     <geometry>
-                      <mesh filename="file:///home/pratik/nala/gazebo_standalone/solo12_robot/solo12_description/meshes/collision/hip_fe_hl.${mesh_ext}"/>
+                      <mesh filename="file:///home/pratik/Music/sdp/solo12_robot/solo12_description/meshes/collision/hip_fe_hl.${mesh_ext}"/>
                     </geometry>
                 </xacro:unless>
@@ -98,5 +98,5 @@
                     <origin xyz="0.01950 0 0" rpy="0 0 0" />
                     <geometry>
-                        <mesh filename="file:///home/pratik/nala/gazebo_standalone/solo12_robot/solo12_description/meshes/collision/hip_fe_fr.${mesh_ext}"/>
+                        <mesh filename="file:///home/pratik/Music/sdp/solo12_robot/solo12_description/meshes/collision/hip_fe_fr.${mesh_ext}"/>
                     </geometry>
                 </xacro:if>
@@ -104,5 +104,5 @@
                     <origin xyz="-0.01950 0 0" rpy="0 0 0" />
                     <geometry>
-                        <mesh filename="file:///home/pratik/nala/gazebo_standalone/solo12_robot/solo12_description/meshes/collision/hip_fe_hr.${mesh_ext}"/>
+                        <mesh filename="file:///home/pratik/Music/sdp/solo12_robot/solo12_description/meshes/collision/hip_fe_hr.${mesh_ext}"/>
                     </geometry>
                 </xacro:unless>
@@ -231,8 +231,8 @@
         <geometry>
           <xacro:unless value="${is_right}">
-            <mesh filename="file:///home/pratik/nala/gazebo_standalone/solo12_robot/solo12_description/meshes/collision/isolated_upper_leg_left_side.${mesh_ext}"/>
-          </xacro:unless>
-          <xacro:if value="${is_right}">
-            <mesh filename="file:///home/pratik/nala/gazebo_standalone/solo12_robot/solo12_description/meshes/collision/isolated_upper_leg_right_side.${mesh_ext}"/>
+            <mesh filename="file:///home/pratik/Music/sdp/solo12_robot/solo12_description/meshes/collision/isolated_upper_leg_left_side.${mesh_ext}"/>
+          </xacro:unless>
+          <xacro:if value="${is_right}">
+            <mesh filename="file:///home/pratik/Music/sdp/solo12_robot/solo12_description/meshes/collision/isolated_upper_leg_right_side.${mesh_ext}"/>
           </xacro:if>
         </geometry>
@@ -246,8 +246,8 @@
         <geometry>
           <xacro:unless value="${is_right}">
-            <mesh filename="file:///home/pratik/nala/gazebo_standalone/solo12_robot/solo12_description/meshes/collision/isolated_upper_leg_left_side.${mesh_ext}"/>
-          </xacro:unless>
-          <xacro:if value="${is_right}">
-            <mesh filename="file:///home/pratik/nala/gazebo_standalone/solo12_robot/solo12_description/meshes/collision/isolated_upper_leg_right_side.${mesh_ext}"/>
+            <mesh filename="file:///home/pratik/Music/sdp/solo12_robot/solo12_description/meshes/collision/isolated_upper_leg_left_side.${mesh_ext}"/>
+          </xacro:unless>
+          <xacro:if value="${is_right}">
+            <mesh filename="file:///home/pratik/Music/sdp/solo12_robot/solo12_description/meshes/collision/isolated_upper_leg_right_side.${mesh_ext}"/>
           </xacro:if>
         </geometry>
@@ -316,8 +316,8 @@
         <geometry>
           <xacro:unless value="${is_right}">
-            <mesh filename="file:///home/pratik/nala/gazebo_standalone/solo12_robot/solo12_description/meshes/collision/isolated_lower_leg_v2_left_side.${mesh_ext}"/>
-          </xacro:unless>
-          <xacro:if value="${is_right}">
-            <mesh filename="file:///home/pratik/nala/gazebo_standalone/solo12_robot/solo12_description/meshes/collision/isolated_lower_leg_v2_right_side.${mesh_ext}"/>
+            <mesh filename="file:///home/pratik/Music/sdp/solo12_robot/solo12_description/meshes/collision/isolated_lower_leg_v2_left_side.${mesh_ext}"/>
+          </xacro:unless>
+          <xacro:if value="${is_right}">
+            <mesh filename="file:///home/pratik/Music/sdp/solo12_robot/solo12_description/meshes/collision/isolated_lower_leg_v2_right_side.${mesh_ext}"/>
           </xacro:if>
         </geometry>
@@ -331,8 +331,8 @@
         <geometry>
           <xacro:unless value="${is_right}">
-            <mesh filename="file:///home/pratik/nala/gazebo_standalone/solo12_robot/solo12_description/meshes/collision/isolated_lower_leg_v2_left_side.${mesh_ext}"/>
-          </xacro:unless>
-          <xacro:if value="${is_right}">
-            <mesh filename="file:///home/pratik/nala/gazebo_standalone/solo12_robot/solo12_description/meshes/collision/isolated_lower_leg_v2_right_side.${mesh_ext}"/>
+            <mesh filename="file:///home/pratik/Music/sdp/solo12_robot/solo12_description/meshes/collision/isolated_lower_leg_v2_left_side.${mesh_ext}"/>
+          </xacro:unless>
+          <xacro:if value="${is_right}">
+            <mesh filename="file:///home/pratik/Music/sdp/solo12_robot/solo12_description/meshes/collision/isolated_lower_leg_v2_right_side.${mesh_ext}"/>
           </xacro:if>
         </geometry>

File: solo12_description/urdf/modified/solo12.urdf (robot description, URDF)
Before this commit: robot solo, 17 links, 16 joints
Links:
- link FL_LOWER_LEG: geometry collision mesh filename=file:///home/pratik/Music/sdp/solo12_robot/solo12_descripti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; visual mesh filename=file:///home/pratik/Music/sdp/solo12_robot/solo12_descripti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
- link FL_SHOULDER: geometry collision mesh filename=file:///home/pratik/Music/sdp/solo12_robot/solo12_descripti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; visual mesh filename=file:///home/pratik/Music/sdp/solo12_robot/solo12_descripti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
- link FL_UPPER_LEG: geometry collision mesh filename=file:///home/pratik/Music/sdp/solo12_robot/solo12_descripti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; visual mesh filename=file:///home/pratik/Music/sdp/solo12_robot/solo12_descripti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
- link FR_LOWER_LEG: geometry collision mesh filename=file:///home/pratik/Music/sdp/solo12_robot/solo12_descripti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; visual mesh filename=file:///home/pratik/Music/sdp/solo12_robot/solo12_descripti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
- link FR_SHOULDER: geometry collision mesh filename=file:///home/pratik/Music/sdp/solo12_robot/solo12_descripti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; visual mesh filename=file:///home/pratik/Music/sdp/solo12_robot/solo12_descripti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
- link FR_UPPER_LEG: geometry collision mesh filename=file:///home/pratik/Music/sdp/solo12_robot/solo12_descripti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; visual mesh filename=file:///home/pratik/Music/sdp/solo12_robot/solo12_descripti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
- link HL_LOWER_LEG: geometry collision mesh filename=file:///home/pratik/Music/sdp/solo12_robot/solo12_descripti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; visual mesh filename=file:///home/pratik/Music/sdp/solo12_robot/solo12_descripti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
- link HL_SHOULDER: geometry collision mesh filename=file:///home/pratik/Music/sdp/solo12_robot/solo12_descripti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; visual mesh filename=file:///home/pratik/Music/sdp/solo12_robot/solo12_descripti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
- link HL_UPPER_LEG: geometry collision mesh filename=file:///home/pratik/Music/sdp/solo12_robot/solo12_descripti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; visual mesh filename=file:///home/pratik/Music/sdp/solo12_robot/solo12_descripti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
- link HR_LOWER_LEG: geometry collision mesh filename=file:///home/pratik/Music/sdp/solo12_robot/solo12_descripti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; visual mesh filename=file:///home/pratik/Music/sdp/solo12_robot/solo12_descripti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
- link HR_SHOULDER: geometry collision mesh filename=file:///home/pratik/Music/sdp/solo12_robot/solo12_descripti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; visual mesh filename=file:///home/pratik/Music/sdp/solo12_robot/solo12_descripti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
- link HR_UPPER_LEG: geometry collision mesh filename=file:///home/pratik/Music/sdp/solo12_robot/solo12_descripti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; visual mesh filename=file:///home/pratik/Music/sdp/solo12_robot/solo12_descripti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
- link base_link: geometry collision mesh filename=file:///home/pratik/Music/sdp/solo12_robot/solo12_descripti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; visual mesh filename=file:///home/pratik/Music/sdp/solo12_robot/solo12_descripti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

File: solo12_description/urdf/modified/solo12.urdf.xacro (robot description, xacro)
@@ -26,5 +26,5 @@
         <geometry>
       <!-- <box size="0.1 0.1 0.1"/>-->
-      <mesh filename="file:///home/pratik/nala/gazebo_standalone/solo12_robot/solo12_description/meshes/collision/base.${mesh_ext}"/>
+      <mesh filename="file:///home/pratik/Music/sdp/solo12_robot/solo12_description/meshes/collision/base.${mesh_ext}"/>
         </geometry>
         <material name="${color_name}">
@@ -36,5 +36,5 @@
         <origin xyz="0 0 0" rpy="0 0 0" />
         <geometry>
-      <mesh filename="file:///home/pratik/nala/gazebo_standalone/solo12_robot/solo12_description/meshes/collision/base.${mesh_ext}"/>
+      <mesh filename="file:///home/pratik/Music/sdp/solo12_robot/solo12_description/meshes/collision/base.${mesh_ext}"/>
         </geometry>
         <material name="${color_name}">
