Commit message: add `use_sim` arguments to allow dynamic interface usage

File: solo12_description/urdf/solo12.ros2_control.xacro (robot description, xacro)
@@ -1,73 +1,88 @@
 <?xml version="1.0" ?>
 <robot xmlns:xacro="http://www.ros.org/wiki/xacro">
-  <ros2_control name="GazeboSystem" type="system">
-    <hardware>
-      <plugin>gazebo_ros2_control/GazeboSystem</plugin>
-    </hardware>
-    <joint name="FL_HAA">
-      <command_interface name="velocity"/>
-      <state_interface name="position"/>
-      <state_interface name="velocity"/>
-    </joint>
-    <joint name="FL_HFE">
-      <command_interface name="velocity"/>
-      <state_interface name="position"/>
-      <state_interface name="velocity"/>
-    </joint>
-    <joint name="FL_KFE">
-      <command_interface name="velocity"/>
-      <state_interface name="position"/>
-      <state_interface name="velocity"/>
-    </joint>
-    <joint name="FR_HAA">
-      <command_interface name="velocity"/>
-      <state_interface name="position"/>
-      <state_interface name="velocity"/>
-    </joint>
-    <joint name="FR_HFE">
-      <command_interface name="velocity"/>
-      <state_interface name="position"/>
-      <state_interface name="velocity"/>
-    </joint>
-    <joint name="FR_KFE">
-      <command_interface name="velocity"/>
-      <state_interface name="position"/>
-      <state_interface name="velocity"/>
-    </joint>
-    <joint name="HL_HAA">
-      <command_interface name="velocity"/>
-      <state_interface name="position"/>
-      <state_interface name="velocity"/>
-    </joint>
-    <joint name="HL_HFE">
-      <command_interface name="velocity"/>
-      <state_interface name="position"/>
-      <state_interface name="velocity"/>
-    </joint>
-    <joint name="HL_KFE">
-      <command_interface name="velocity"/>
-      <state_interface name="position"/>
-      <state_interface name="velocity"/>
-    </joint>
-    <joint name="HR_HAA">
-      <command_interface name="velocity"/>
-      <state_interface name="position"/>
-      <state_interface name="velocity"/>
-    </joint>
-    <joint name="HR_HFE">
-      <command_interface name="velocity"/>
-      <state_interface name="position"/>
-      <state_interface name="velocity"/>
-    </joint>
-    <joint name="HR_KFE">
-      <command_interface name="velocity"/>
-      <state_interface name="position"/>
-      <state_interface name="velocity"/>
-    </joint>
-  </ros2_control>
-  <gazebo>
-    <plugin name="gazebo_ros2_control" filename="libgazebo_ros2_control.so">
-      <parameters>$(find solo12_description)/config/solo12_controllers.yaml</parameters>
-    </plugin>
-  </gazebo>
+  <xacro:macro name="solo12_ros2_control" params="use_sim">
+      <ros2_control name="Solo12HardwareInterface" type="system">
+        <hardware>
+          <!-- If "use_sim" argument is set to true launch gazebo simulation -->
+          <xacro:if value="${use_sim}">
+            <plugin>gazebo_ros2_control/GazeboSystem</plugin>
+          </xacro:if>
+          <!--
+            Otherwise launch real hardware
+          TODO:
+          - add hardware interface for the robot
+          -->
+          <xacro:unless value="${use_sim}">
+            <plugin>placeholder_namespace/PlaceHolderClass</plugin>
+          </xacro:unless>
+        </hardware>
+        <joint name="FL_HAA">
+          <command_interface name="velocity"/>
+          <state_interface name="position"/>
+          <state_interface name="velocity"/>
+        </joint>
+        <joint name="FL_HFE">
+          <command_interface name="velocity"/>
+          <state_interface name="position"/>
+          <state_interface name="velocity"/>
+        </joint>
+        <joint name="FL_KFE">
+          <command_interface name="velocity"/>
+          <state_interface name="position"/>
+          <state_interface name="velocity"/>
+        </joint>
+        <joint name="FR_HAA">
+          <command_interface name="velocity"/>
+          <state_interface name="position"/>
+          <state_interface name="velocity"/>
+        </joint>
+        <joint name="FR_HFE">
+          <command_interface name="velocity"/>
+          <state_interface name="position"/>
+          <state_interface name="velocity"/>
+        </joint>
+        <joint name="FR_KFE">
+          <command_interface name="velocity"/>
+          <state_interface name="position"/>
+          <state_interface name="velocity"/>
+        </joint>
+        <joint name="HL_HAA">
+          <command_interface name="velocity"/>
+          <state_interface name="position"/>
+          <state_interface name="velocity"/>
+        </joint>
+        <joint name="HL_HFE">
+          <command_interface name="velocity"/>
+          <state_interface name="position"/>
+          <state_interface name="velocity"/>
+        </joint>
+        <joint name="HL_KFE">
+          <command_interface name="velocity"/>
+          <state_interface name="position"/>
+          <state_interface name="velocity"/>
+        </joint>
+        <joint name="HR_HAA">
+          <command_interface name="velocity"/>
+          <state_interface name="position"/>
+          <state_interface name="velocity"/>
+        </joint>
+        <joint name="HR_HFE">
+          <command_interface name="velocity"/>
+          <state_interface name="position"/>
+          <state_interface name="velocity"/>
+        </joint>
+        <joint name="HR_KFE">
+          <command_interface name="velocity"/>
+          <state_interface name="position"/>
+          <state_interface name="velocity"/>
+        </joint>
+      </ros2_control>
+    <xacro:if value="${use_sim}">
+      <gazebo>
+        <plugin name="gazebo_ros2_control" filename="libgazebo_ros2_control.so">
+          <parameters>$(find solo12_description)/config/solo12_controllers.yaml</parameters>
+        </plugin>
+      </gazebo>
+    </xacro:if>
+  </xacro:macro>
 </robot>

File: solo12_description/urdf/solo12.urdf.xacro (robot description, xacro)
@@ -5,4 +5,5 @@
   xmlns:sensor="http://playerstage.sourceforge.net/gazebo/xmlschema/#sensor"
   xmlns:xacro="http://playerstage.sourceforge.net/gazebo/xmlschema/#interface">
+  <xacro:arg name="use_sim" default="true" />
   <xacro:property name="color_name" value="grey" />
   <xacro:property name="color" value="0.8 0.8 0.8" />
@@ -10,4 +11,6 @@
   <xacro:property name="mesh_ext" value="stl" />
   <xacro:include filename="solo12.ros2_control.xacro"/>
+  <xacro:solo12_ros2_control
+    use_sim="$(arg use_sim)"/>
   <!-- This file is based on: https://github.com/open-dynamic-robot-initiative/open_robot_actuator_hardware/blob/master/mechanics/quadruped_robot_12dof_v1/README.md#quadruped-robot-12dof-v1 -->
   <link name="base_link">

Commit message: add robot network interface for communication

File: solo12_description/urdf/solo12.ros2_control.xacro (robot description, xacro)
@@ -1,5 +1,8 @@
 <?xml version="1.0" ?>
 <robot xmlns:xacro="http://www.ros.org/wiki/xacro">
-  <xacro:macro name="solo12_ros2_control" params="use_sim">
+  <xacro:macro name="solo12_ros2_control" params="
+    use_sim:=true
+    robot_interface:=enp1s0
+    ">
       <ros2_control name="Solo12HardwareInterface" type="system">
         <hardware>
@@ -11,4 +14,5 @@
           <xacro:unless value="${use_sim}">
             <plugin>solo12_hardware_interface/Solo12HardwareInterface</plugin>
+            <param name="robot_interface">${robot_interface}</param>
           </xacro:unless>
         </hardware>
